File: nfc.kicad_sch (KiCad schematic)
At the start: 16 parts, among them Y1 Crystal_GND24

Commit message: Almost finalize schematics
Parts:
- removed AE1: Antenna_Loop, symbol Device:Antenna_Loop
- added C30: 100nF, Capacitor_SMD:C_0603_1608Metric, symbol Device:C
- added Cemc2: C, Capacitor_SMD:C_0603_1608Metric, symbol Device:C
- added Cp2: 220p, Capacitor_SMD:C_0603_1608Metric, symbol Device:C
- added Cs2: 78p, Capacitor_SMD:C_0603_1608Metric, symbol Device:C
- added Cvdr3: 212p, Capacitor_SMD:C_0603_1608Metric, symbol Device:C
- added Cvdr4: 10p, Capacitor_SMD:C_0603_1608Metric, symbol Device:C
- added L3: 270nH, Inductor_SMD:L_1210_3225Metric, symbol _GRZ_Passive:INDUCTOR
- added R48: 1.6?, _Resistors_GRZ:R_0603, symbol Device:R
- added R49, R50: 0, _Resistors_GRZ:R_0603, symbol Device:R
- added R7 (x6): 0, Resistor_SMD:R_0603_1608Metric, symbol Device:R
- added TP1, TP2, TP3, TP4, TP5: TestPoint, TestPoint:TestPoint_Pad_D2.0mm, symbol Connector:TestPoint
- added U7: ~, myFootprints:NFC_antenna, symbol mySymbols:NFC_antenna
- L2: value INDUCTOR -> 270nH; footprint (none) -> Inductor_SMD:L_1210_3225Metric
- R35: footprint (none) -> _Resistors_GRZ:R_0603
Connections:
- net +3.3V: now also R7.1; no longer U?.1 (VDD_IO), U?.8 (VDD)
- net GND: now also Cvdr2.2, C30.2, Cemc2.1, Cp2.1, Cvdr3.2; no longer Cvdr2.1
- net NFC_CLK: now also R7.1, TP3.1; no longer U?.31 (SCLK)
- net NFC_IRQ: now also R7.1, TP5.1; no longer U?.27 (IRQ)
- net NFC_MISO: now also R7.1, TP1.1; no longer U?.29 (MISO)
- net NFC_MOSI: now also R7.1, TP2.1; no longer U?.30 (MOSI)
- net NFC_SS: now also R7.1, TP4.1; no longer U?.32 (/SS)
- net RFI1: now also Cvdr1.2, Cvdr2.1; no longer Cvdr1.1, Cvdr2.2
- net at Cp1.2, Cs1.1, R35.1: now also Cvdr1.1; no longer Cvdr1.2
- net RFO2: now reaches U?.11 (RFO2)
- net RFO2: now also L3.1
- net CSO: now reaches U?.2 (CSO)
- net CSO: now also R50.1
- net RFI2: now reaches U?.23 (RFI2)
- net RFI2: now also Cvdr3.1, Cvdr4.2
- net CSI: now reaches U?.25 (CSI)
- net CSI: now also R49.2
- net at R35.2: now also U7.1
- new net: R7.2, U?.30 (MOSI)
- new net: R49.1, U7.3
- new net: C30.1, R7.2, U?.1 (VDD_IO), U?.8 (VDD)
- new net: R7.2, U?.27 (IRQ)
- new net: R7.2, U?.29 (MISO)
- new net: R7.2, U?.31 (SCLK)
- new net: R7.2, U?.32 (/SS)
- new net: Cp2.2, Cs2.1, Cvdr4.1, R48.1
- new net: Cemc2.2, Cs2.2, L3.2
- new net: R50.2, U7.1
- new net: R48.2, U7.2
- no-connect marks 13 -> 9
Other:
- moved on the sheet: C13, C14, C15, C16, C17, C18, Cemc1, Cp1, Cs1, Cvdr1, Cvdr2, L2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

Commit message: Finish layout.
Parts:
- removed R7 (x5): 0, Resistor_SMD:R_0603_1608Metric, symbol Device:R
- removed TP1, TP2, TP3, TP4, TP5: TestPoint, TestPoint:TestPoint_Pad_D2.0mm, symbol Connector:TestPoint
- removed U7: ~, myFootprints:NFC_antenna, symbol mySymbols:NFC_antenna
- added #A1: ~, myFootprints:NFC_antenna, symbol mySymbols:NFC_antenna
- added #J5: Conn_01x07_Pin, _Connectors_GRZ:PicoBlade_53261-0771, symbol Connector:Conn_01x07_Pin
- renumbered C13 to #C13, C14 to #C14, C15 to #C15, C16 to #C16, C17 to #C17, C18 to #C18, C30 to #C30, Cemc1 to #Cemc1, Cemc2 to #Cemc2, Cp1 to #Cp1, Cp2 to #Cp2, Cs1 to #Cs1, Cs2 to #Cs2, Cvdr1 to #Cvdr1, Cvdr2 to #Cvdr2, Cvdr3 to #Cvdr3, Cvdr4 to #Cvdr4, L2 to #L2, L3 to #L3, R35 to #R35, R48 to #R48, R49 to #R49, R50 to #R50, Y1 to #Y1
Connections:
- net +3.3V: now also #J5.2 (Pin_2)
- net GND: now also #J5.1 (Pin_1)
- net MOSI: now reaches U?.30 (MOSI)
- net MOSI: now also #J5.4 (Pin_4)
- net at #R49.1: now also #A1.3
- net IRQ: now reaches U?.27 (IRQ)
- net IRQ: now also #J5.7 (Pin_7)
- net MISO: now reaches U?.29 (MISO)
- net MISO: now also #J5.5 (Pin_5)
- net CLK: now reaches U?.31 (SCLK)
- net CLK: now also #J5.6 (Pin_6)
- net CS: now reaches U?.32 (/SS)
- net CS: now also #J5.3 (Pin_3)
- net at #R35.2: now also #A1.1
- net at #R50.2: now also #A1.4
- net at #R48.2: now also #A1.2
Other:
- moved on the sheet: R7, U?
