File: power_supply.kicad_sch (KiCad schematic)
At the start: 38 parts

Commit message: Almost finalize schematics
Parts:
- removed R?: 1.8kΩ, _Resistors_GRZ:R_0603, symbol _GRZ_Passive:RES1
- removed R?: 3.3kΩ, _Resistors_GRZ:R_0603, symbol _GRZ_Passive:RES1
- added BT2: Battery_Cell, Battery:BatteryHolder_Keystone_3002_1x2032, symbol Device:Battery_Cell
- C? (x4): footprint (none) -> _Capacitors_GRZ:C_0603
- JP1: footprint (none) -> Jumper:SolderJumper-2_P1.3mm_Open_TrianglePad1.0x1.5mm
Connections:
- net GND: now also BT2.2 (-)
- net VBAT: now also BT2.1 (+)
- net +5VUSB renamed USB_VBUS
Other:
- note removed: "TODO change to USB-C"

Commit message: Finish layout.
Parts:
- removed PB?: FSMxJSM, _Switches_GRZ:FSM2JSM, symbol _GRZ_Switches:FSMxJSM
- added PB6: KSC3J, _Switches_GRZ:KSC3J, symbol _GRZ_Switches:KSC3J
Connections:
- net GND: now also BT?.2 (-), PB6.1, PB6.4; no longer BT?.1 (-)
- net POWER_KEY: now also PB6.2, PB6.3
- net VBAT: now also BT?.1 (+); no longer BT2.1 (+), BT?.2 (+)
- new net +BATT: BT2.1 (+)
Changed lines of the file:
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@@
 (kicad_sch (version 20230121) (generator eeschema)
   (paper "A4")
+  (junction (at 196.85 140.97) (diameter 0) (color 0 0 0 0)
+  )
+  (junction (at 246.38 68.58) (diameter 0) (color 0 0 0 0)
+  )
+  (junction (at 53.34 172.72) (diameter 0) (color 0 0 0 0)
+  )
+  (junction (at 27.94 48.26) (diameter 0) (color 0 0 0 0)
+  )
+  (junction (at 147.32 48.26) (diameter 0) (color 0 0 0 0)
+  )
   (junction (at 162.56 87.63) (diameter 0) (color 0 0 0 0)
-  )
-  (junction (at 196.85 140.97) (diameter 0) (color 0 0 0 0)
-  )
-  (junction (at 246.38 68.58) (diameter 0) (color 0 0 0 0)
-  )
-  (junction (at 53.34 172.72) (diameter 0) (color 0 0 0 0)
-  )
-  (junction (at 27.94 48.26) (diameter 0) (color 0 0 0 0)
-  )
-  (junction (at 147.32 48.26) (diameter 0) (color 0 0 0 0)
   )
   (junction (at 210.82 130.81) (diameter 0) (color 0 0 0 0)
@@
     )
   )
-  (symbol (lib_id "_GRZ_Switches:FSMxJSM") (at 162.56 85.09 90) (unit 1)
-    (in_bom yes) (on_board yes) (dnp no)
-    (property "Reference" "PB?" (at 149.86 82.55 90)
-      (effects (font (size 1.27 1.27)) (justify right))
-    )
-    (property "Value" "FSMxJSM" (at 147.32 85.09 90)
-      (effects (font (size 1.27 1.27)) (justify right))
-    )
-    (property "Footprint" "_Switches_GRZ:FSM2JSM" (at 165.1 85.09 0)
-      (effects (font (size 1.27 1.27)) hide)
-    )
-    (property "Datasheet" "" (at 157.48 83.82 0)
-      (effects (font (size 1.27 1.27)) hide)
-    )
-    (pin "1")
-    (pin "3")
-    (pin "2")
-    (pin "4")
-    (instances
-      (project ""
-        (path "/6441b183-b8f2-458f-a23d-60e2b1f66dd6"
-          (reference "PB?") (unit 1)
-        )
-      )
-      (project "battery_tester"
-        (path "/f5c3540e-6306-4c42-9ce5-3ef8f6308672/654b8b52-3828-4936-bf17-3bb11f963210"
-          (reference "PB5") (unit 1)
-        )
-      )
-    )
-  )
   (symbol (lib_id "power:PWR_FLAG") (at 71.12 35.56 0) (unit 1)
     (in_bom yes) (on_board yes) (dnp no) (fields_autoplaced)
@@
     )
   )
-  (symbol (lib_id "_GRZ_Power:VBAT") (at 27.94 46.99 0) (unit 1)
-    (in_bom yes) (on_board yes) (dnp no)
-    (property "Reference" "#PWR098" (at 27.94 48.895 0)
-      (effects (font (size 1.27 1.27)) hide)
-    )
-    (property "Value" "VBAT" (at 27.94 43.18 0)
-      (effects (font (size 1.27 1.27)))
-    )
-    (property "Footprint" "" (at 27.94 46.99 0)
-      (effects (font (size 1.27 1.27)) hide)
-    )
-    (property "Datasheet" "" (at 27.94 46.99 0)
-      (effects (font (size 1.27 1.27)) hide)
-    )
-    (pin "1")
-    (instances
-      (project "battery_tester"
-        (path "/f5c3540e-6306-4c42-9ce5-3ef8f6308672"
-          (reference "#PWR098") (unit 1)
-        )
-        (path "/f5c3540e-6306-4c42-9ce5-3ef8f6308672/654b8b52-3828-4936-bf17-3bb11f963210"
-          (reference "#PWR097") (unit 1)
-        )
-      )
-    )
-  )
   (symbol (lib_id "Device:C") (at 215.9 137.16 0) (unit 1)
     (in_bom yes) (on_board yes) (dnp no)
@@
     )
   )
+  (symbol (lib_id "power:+BATT") (at 27.94 46.99 0) (unit 1)
+    (in_bom yes) (on_board yes) (dnp no) (fields_autoplaced)
+    (property "Reference" "#PWR097" (at 27.94 50.8 0)
+      (effects (font (size 1.27 1.27)) hide)
+    )
+    (property "Value" "+BATT" (at 27.94 41.91 0)
+      (effects (font (size 1.27 1.27)))
+    )
+    (property "Footprint" "" (at 27.94 46.99 0)
+      (effects (font (size 1.27 1.27)) hide)
+    )
+    (property "Datasheet" "" (at 27.94 46.99 0)
+      (effects (font (size 1.27 1.27)) hide)
+    )
+    (pin "1")
+    (instances
+      (project "battery_tester"
+        (path "/f5c3540e-6306-4c42-9ce5-3ef8f6308672/654b8b52-3828-4936-bf17-3bb11f963210"
+          (reference "#PWR097") (unit 1)
+        )
+      )
+    )
+  )
   (symbol (lib_id "power:+3.3V") (at 219.71 130.81 270) (unit 1)
     (in_bom yes) (on_board yes) (dnp no) (fields_autoplaced)
@@
         )
       )
+    )
+  )
+  (symbol (lib_id "_GRZ_Switches:KSC3J") (at 162.56 85.09 90) (unit 1)
+    (in_bom yes) (on_board yes) (dnp no)
+    (property "Reference" "PB6" (at 157.48 87.63 0)
+      (effects (font (size 1.27 1.27)))
+    )
+    (property "Value" "KSC3J" (at 157.48 78.74 0)
+      (effects (font (size 1.27 1.27)))
+    )
+    (property "Footprint" "_Switches_GRZ:KSC3J" (at 165.1 85.09 0)
+      (effects (font (size 1.27 1.27)) hide)
+    )
+    (property "Datasheet" "" (at 157.48 83.82 0)
+      (effects (font (size 1.27 1.27)) hide)
+    )
+    (pin "3")
+    (pin "4")
+    (pin "1")
+    (pin "2")
+    (instances
+      (project "battery_tester"
+        (path "/f5c3540e-6306-4c42-9ce5-3ef8f6308672"
+          (reference "PB6") (unit 1)
+        )
+        (path "/f5c3540e-6306-4c42-9ce5-3ef8f6308672/654b8b52-3828-4936-bf17-3bb11f963210"
+          (reference "PB7") (unit 1)
+        )
+      )
